File: mcu.kicad_sch (KiCad schematic)
At the start: 11 parts, among them U1 ATMEGA8A-AN, Y1 CSTNE16M0V530000R0

Commit message: Do PCB
Parts:
- removed U1: ATMEGA8A-AN, U_IC:LQFP32_08_7x7, symbol U_MCU:ATMEGA8A-AN
- added U1: ATMEGA8A-MU, U_IC:QFN32_05_5x5_EP, symbol U_MCU:ATMEGA8A-MU
Connections:
- net +5V: now also U1.18 (AVCC), U1.20 (AREF), U1.4 (VCC), U1.6 (VCC)
- net GND: now also U1.21 (GND), U1.3 (GND), U1.33 (EP), U1.5 (GND)
- net ICSP_NRST: now also U1.29 (NRST/PC5)
- net MISO: now also U1.16 (PB4/MISO)
- net MOSI: now also U1.15 (PB3/MOSI)
- net NRST: now also U1.14 (PB2)
- net RX: now also U1.30 (RXD/PD0)
- net SCK: now also U1.17 (SCK/PB5)
- net TX: now also U1.31 (TXD/PD1)
- net at Y1.1: now also U1.7 (PB7/XTAL1)
- net at Y1.3: now also U1.8 (PB7/XTAL2)

Commit message: Fix direction issue on MISO/MOSI
Changed lines of the file:
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@@
     (effects (font (size 1.27 1.27)) (justify left))
   )
-  (hierarchical_label "RX" (shape output) (at 128.27 31.75 90) (fields_autoplaced)
+  (hierarchical_label "RX" (shape input) (at 128.27 31.75 90) (fields_autoplaced)
     (effects (font (size 1.27 1.27)) (justify left))
   )
