File: target.kicad_sch (KiCad schematic)
At the start: 1 part, among them J2 61200621621

Commit message: Do PCB
Parts:
- added J3: Pins_2.54_1x2, J_Connector:Pins-2.54-1x2, symbol J_Connector:Pins_2.54_1x2
- added U3, U4, U5, U6: 74LVC1T45Z6, U_IC:SOT563, symbol U_Basic:74LVC1T45Z6
Connections:
- net GND: now also J3.2, U3.2 (GND), U3.5 (DIR), U4.2 (GND), U5.2 (GND), U5.5 (DIR), U6.2 (GND), U6.5 (DIR)
- net MISO: now also U5.4 (B); no longer J2.1 (Pin_1)
- net MOSI: now also U4.4 (B); no longer J2.4 (Pin_4)
- net NRST: now also U6.4 (B); no longer J2.5 (Pin_5)
- net SCK: now also U3.4 (B); no longer J2.3 (Pin_3)
- net TARGET_VCC: now also J3.1, U3.1 (VCCA), U4.1 (VCCA), U5.1 (VCCA), U6.1 (VCCA)
- new net +5V: U3.6 (VCCB), U4.5 (DIR), U4.6 (VCCB), U5.6 (VCCB), U6.6 (VCCB)
- new net TARGET_MISO: J2.1 (Pin_1), U5.3 (A)
- new net TARGET_MOSI: J2.4 (Pin_4), U4.3 (A)
- new net TARGET_NRST: J2.5 (Pin_5), U6.3 (A)
- new net TARGET_SCK: J2.3 (Pin_3), U3.3 (A)
Other:
- note removed: "ATMEGA8A-MU"
- note removed: "PCA9306"
- moved on the sheet: J2

Commit message: Update readme
Add jumper to tie 5V to VCC
Parts:
- added JP1: SolderJumper2, Jumper:SolderJumper-2_P1.3mm_Open_RoundedPad1.0x1.5mm, symbol Jumper:SolderJumper_2_Open
Connections:
- net +5V: now also JP1.1 (A)
- net TARGET_VCC: now also JP1.2 (B)
Other:
- moved on the sheet: J3
Changed lines of the file:
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@@
     (stroke (width 0) (type default))
   )
-  (wire (pts (xy 142.24 86.36) (xy 142.24 83.82))
+  (wire (pts (xy 171.45 91.44) (xy 171.45 88.9))
     (stroke (width 0) (type default))
   )
@@
     (stroke (width 0) (type default))
   )
+  (wire (pts (xy 137.16 86.36) (xy 143.51 86.36))
+    (stroke (width 0) (type default))
+  )
   (wire (pts (xy 86.36 69.85) (xy 91.44 69.85))
     (stroke (width 0) (type default))
@@
     (stroke (width 0) (type default))
   )
-  (wire (pts (xy 142.24 83.82) (xy 144.78 83.82))
+  (wire (pts (xy 171.45 88.9) (xy 173.99 88.9))
     (stroke (width 0) (type default))
   )
@@
     (stroke (width 0) (type default))
   )
+  (wire (pts (xy 137.16 85.09) (xy 137.16 86.36))
+    (stroke (width 0) (type default))
+  )
   (wire (pts (xy 86.36 66.04) (xy 105.41 66.04))
     (stroke (width 0) (type default))
   )
-  (wire (pts (xy 130.81 81.28) (xy 144.78 81.28))
+  (wire (pts (xy 151.13 86.36) (xy 173.99 86.36))
     (stroke (width 0) (type default))
   )
@@
     (effects (font (size 1.27 1.27)) (justify right bottom))
   )
-  (label "TARGET_VCC" (at 130.81 81.28 0) (fields_autoplaced)
+  (label "TARGET_VCC" (at 160.02 86.36 0) (fields_autoplaced)
     (effects (font (size 1.27 1.27)) (justify left bottom))
   )
@@
         (path "/5952f252-dd2a-4213-9849-5d3ec960c0f2/503087ff-ef98-4ee3-b2a9-012004e0bc0f"
           (reference "#PWR026") (unit 1)
+        )
+      )
+    )
+  )
+  (symbol (lib_id "power:+5V") (at 137.16 85.09 0) (unit 1)
+    (in_bom yes) (on_board yes) (dnp no) (fields_autoplaced)
+    (property "Reference" "#PWR037" (at 137.16 88.9 0)
+      (effects (font (size 1.27 1.27)) hide)
+    )
+    (property "Value" "+5V" (at 137.16 81.5881 0)
+      (effects (font (size 1.27 1.27)))
+    )
+    (property "Footprint" "" (at 137.16 85.09 0)
+      (effects (font (size 1.27 1.27)) hide)
+    )
+    (property "Datasheet" "" (at 137.16 85.09 0)
+      (effects (font (size 1.27 1.27)) hide)
+    )
+    (pin "1")
+    (instances
+      (project "ICSP-Programmer-HW"
+        (path "/5952f252-dd2a-4213-9849-5d3ec960c0f2/503087ff-ef98-4ee3-b2a9-012004e0bc0f"
+          (reference "#PWR037") (unit 1)
         )
       )
@@
     )
   )
-  (symbol (lib_id "power:GND") (at 142.24 86.36 0) (unit 1)
+  (symbol (lib_id "power:GND") (at 171.45 91.44 0) (unit 1)
     (in_bom yes) (on_board yes) (dnp no)
-    (property "Reference" "#PWR027" (at 142.24 92.71 0)
-      (effects (font (size 1.27 1.27)) hide)
-    )
-    (property "Value" "GND" (at 142.24 93.98 90)
+    (property "Reference" "#PWR027" (at 171.45 97.79 0)
+      (effects (font (size 1.27 1.27)) hide)
+    )
+    (property "Value" "GND" (at 171.45 99.06 90)
       (effects (font (size 1.27 1.27)) (justify left))
     )
-    (property "Footprint" "" (at 142.24 86.36 0)
-      (effects (font (size 1.27 1.27)) hide)
-    )
-    (property "Datasheet" "" (at 142.24 86.36 0)
+    (property "Footprint" "" (at 171.45 91.44 0)
+      (effects (font (size 1.27 1.27)) hide)
+    )
+    (property "Datasheet" "" (at 171.45 91.44 0)
       (effects (font (size 1.27 1.27)) hide)
     )
@@
     )
   )
+  (symbol (lib_id "Jumper:SolderJumper_2_Open") (at 147.32 86.36 0) (unit 1)
+    (in_bom yes) (on_board yes) (dnp no) (fields_autoplaced)
+    (property "Reference" "JP1" (at 147.32 82.4611 0)
+      (effects (font (size 1.27 1.27)))
+    )
+    (property "Value" "SolderJumper2" (at 147.32 84.3821 0)
+      (effects (font (size 1.27 1.27)))
+    )
+    (property "Footprint" "Jumper:SolderJumper-2_P1.3mm_Open_RoundedPad1.0x1.5mm" (at 147.32 86.36 0)
+      (effects (font (size 1.27 1.27)) hide)
+    )
+    (property "Datasheet" "~" (at 147.32 86.36 0)
+      (effects (font (size 1.27 1.27)) hide)
+    )
+    (pin "1")
+    (pin "2")
+    (instances
+      (project "ICSP-Programmer-HW"
+        (path "/5952f252-dd2a-4213-9849-5d3ec960c0f2/503087ff-ef98-4ee3-b2a9-012004e0bc0f"
+          (reference "JP1") (unit 1)
+        )
+      )
+    )
+  )
   (symbol (lib_id "power:+5V") (at 63.5 34.29 0) (unit 1)
     (in_bom yes) (on_board yes) (dnp no) (fields_autoplaced)
@@
     )
   )
-  (symbol (lib_id "J_Connector:Pins_2.54_1x2") (at 148.59 85.09 0) (unit 1)
-    (in_bom yes) (on_board yes) (dnp no) (fields_autoplaced)
-    (property "Reference" "J3" (at 150.5712 81.9063 0)
+  (symbol (lib_id "J_Connector:Pins_2.54_1x2") (at 177.8 90.17 0) (unit 1)
+    (in_bom yes) (on_board yes) (dnp no) (fields_autoplaced)
+    (property "Reference" "J3" (at 179.7812 86.9863 0)
       (effects (font (size 1.27 1.27)) (justify left))
     )
-    (property "Value" "Pins_2.54_1x2" (at 150.5712 83.8273 0)
+    (property "Value" "Pins_2.54_1x2" (at 179.7812 88.9073 0)
       (effects (font (size 1.27 1.27)) (justify left))
     )
-    (property "Footprint" "J_Connector:Pins-2.54-1x2" (at 148.59 88.265 0)
-      (effects (font (size 1.27 1.27)) hide)
-    )
-    (property "Datasheet" "" (at 148.59 85.09 0)
-      (effects (font (size 1.27 1.27)) hide)
-    )
+    (property "Footprint" "J_Connector:Pins-2.54-1x2" (at 177.8 93.345 0)
+      (effects (font (size 1.27 1.27)) hide)
+    )
+    (property "Datasheet" "" (at 177.8 90.17 0)
+      (effects (font (size 1.27 1.27)) hide)
+    )

Commit message: Fix direction issue on MISO/MOSI
Connections:
- net +5V: now also U5.5 (DIR); no longer U4.5 (DIR)
- net GND: now also U4.5 (DIR); no longer U5.5 (DIR)
Changed lines of the file:
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@@
     (effects (font (size 1.27 1.27)) (justify right))
   )
-  (symbol (lib_name "GND_1") (lib_id "power:GND") (at 60.96 91.44 270) (unit 1)
-    (in_bom yes) (on_board yes) (dnp no) (fields_autoplaced)
-    (property "Reference" "#PWR029" (at 54.61 91.44 0)
-      (effects (font (size 1.27 1.27)) hide)
-    )
-    (property "Value" "GND" (at 57.7851 91.7568 90)
-      (effects (font (size 1.27 1.27)) (justify right))
-    )
-    (property "Footprint" "" (at 60.96 91.44 0)
-      (effects (font (size 1.27 1.27)) hide)
-    )
-    (property "Datasheet" "" (at 60.96 91.44 0)
-      (effects (font (size 1.27 1.27)) hide)
-    )
-    (pin "1")
-    (instances
-      (project "ICSP-Programmer-HW"
-        (path "/5952f252-dd2a-4213-9849-5d3ec960c0f2/503087ff-ef98-4ee3-b2a9-012004e0bc0f"
-          (reference "#PWR029") (unit 1)
-        )
-      )
-    )
-  )
   (symbol (lib_name "GND_1") (lib_id "power:GND") (at 91.44 118.11 0) (unit 1)
     (in_bom yes) (on_board yes) (dnp no) (fields_autoplaced)
@@
         (path "/5952f252-dd2a-4213-9849-5d3ec960c0f2/503087ff-ef98-4ee3-b2a9-012004e0bc0f"
           (reference "#PWR037") (unit 1)
-        )
-      )
-    )
-  )
-  (symbol (lib_id "power:+5V") (at 60.96 69.85 90) (unit 1)
-    (in_bom yes) (on_board yes) (dnp no) (fields_autoplaced)
-    (property "Reference" "#PWR031" (at 64.77 69.85 0)
-      (effects (font (size 1.27 1.27)) hide)
-    )
-    (property "Value" "+5V" (at 57.7851 70.1668 90)
-      (effects (font (size 1.27 1.27)) (justify left))
-    )
-    (property "Footprint" "" (at 60.96 69.85 0)
-      (effects (font (size 1.27 1.27)) hide)
-    )
-    (property "Datasheet" "" (at 60.96 69.85 0)
-      (effects (font (size 1.27 1.27)) hide)
-    )
-    (pin "1")
-    (instances
-      (project "ICSP-Programmer-HW"
-        (path "/5952f252-dd2a-4213-9849-5d3ec960c0f2/503087ff-ef98-4ee3-b2a9-012004e0bc0f"
-          (reference "#PWR031") (unit 1)
         )
       )
@@
     )
   )
+  (symbol (lib_name "GND_1") (lib_id "power:GND") (at 60.96 69.85 270) (unit 1)
+    (in_bom yes) (on_board yes) (dnp no) (fields_autoplaced)
+    (property "Reference" "#PWR029" (at 54.61 69.85 0)
+      (effects (font (size 1.27 1.27)) hide)
+    )
+    (property "Value" "GND" (at 57.7851 70.1668 90)
+      (effects (font (size 1.27 1.27)) (justify right))
+    )
+    (property "Footprint" "" (at 60.96 69.85 0)
+      (effects (font (size 1.27 1.27)) hide)
+    )
+    (property "Datasheet" "" (at 60.96 69.85 0)
+      (effects (font (size 1.27 1.27)) hide)
+    )
+    (pin "1")
+    (instances
+      (project "ICSP-Programmer-HW"
+        (path "/5952f252-dd2a-4213-9849-5d3ec960c0f2/503087ff-ef98-4ee3-b2a9-012004e0bc0f"
+          (reference "#PWR029") (unit 1)
+        )
+      )
+    )
+  )
   (symbol (lib_id "power:GND") (at 171.45 91.44 0) (unit 1)
     (in_bom yes) (on_board yes) (dnp no)
@@
         )
       )
+    )
+  )
+  (symbol (lib_id "power:+5V") (at 60.96 91.44 90) (unit 1)
+    (in_bom yes) (on_board yes) (dnp no) (fields_autoplaced)
+    (property "Reference" "#PWR031" (at 64.77 91.44 0)
+      (effects (font (size 1.27 1.27)) hide)
+    )
+    (property "Value" "+5V" (at 57.7851 91.7568 90)
+      (effects (font (size 1.27 1.27)) (justify left))
+    )
+    (property "Footprint" "" (at 60.96 91.44 0)
+      (effects (font (size 1.27 1.27)) hide)
+    )
+    (property "Datasheet" "" (at 60.96 91.44 0)
+      (effects (font (size 1.27 1.27)) hide)
+    )
+    (pin "1")
+    (instances
+      (project "ICSP-Programmer-HW"
+        (path "/5952f252-dd2a-4213-9849-5d3ec960c0f2/503087ff-ef98-4ee3-b2a9-012004e0bc0f"
+          (reference "#PWR031") (unit 1)
+        )
+      )
