File: usb.kicad_sch (KiCad schematic)
At the start: 10 parts, among them J1 USB4105-GF-A-060, U2 FT230XQ

Commit message: Fix direction issue on MISO/MOSI
Changed lines of the file:
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@@
     (effects (font (size 1.27 1.27)) (justify left))
   )
-  (hierarchical_label "RX" (shape output) (at 205.74 68.58 0) (fields_autoplaced)
+  (hierarchical_label "RX" (shape input) (at 205.74 68.58 0) (fields_autoplaced)
     (effects (font (size 1.27 1.27)) (justify left))
   )
